File: pcb-v2/pcb-v2.kicad_sch (KiCad schematic)
At the start: 47 parts, among them J1 USB_C_Receptacle_USB2.0, J2 USB_A, J3 Conn_01x05, J3 USB_A, SW1 SW_Push, SW2 SW_Push, U1 SRV05-4, U2 SRV05-4, U3 SRV05-4, U4 RP2040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

Commit message: feat: attempt at using ch334
Parts:
- removed C1, C19: 10u, symbol Device:C_Small
- removed C2: 100n, symbol Device:C_Small
- removed R3: 2k7, symbol Device:R_Small
- removed R4: 10k, symbol Device:R_Small
- removed R5: 47k, symbol Device:R_Small
- removed R6: 100k, symbol Device:R_Small
- removed R7: 20k, symbol Device:R_Small
- removed U1, U2, U3: SRV05-4, PCM_marbastlib-various:SOT-23-6-routable, symbol PCM_marbastlib-various:SRV05-4
- removed U5: FE1.1s-BSOP28BPTR, Package_SO:SSOP-28_3.9x9.9mm_P0.635mm, symbol Custom:FE1.1s-BSOP28BPTR
- added C20: 10u, symbol Device:C_Small
- added C21: 0.1u, symbol Device:C_Small
- added C22, C23: 1uF, symbol Device:C_Small
- added R14: 10k, symbol Device:R_Small
- added U8: CH217K, Package_TO_SOT_SMD:SOT-23-6, symbol Custom:CH217K
- added U9: CH334U, Package_SO:SSOP-28_3.9x9.9mm_P0.635mm, symbol Custom:CH334U
Connections:
- net +3V3: now also C20.1, C21.1, C22.1, U9.13 (VDD33), U9.21 (VDD33)
- net +5V: now also C23.1, U9.20 (V5)
- net DM1: now also U9.10 (DM1)
- net DM2: now also U9.8 (DM2)
- net DM3: now also U9.6 (DM3)
- net DMU: now also U9.15 (DMU)
- net DP1: now also U9.11 (DP1)
- net DP2: now also U9.9 (DP2)
- net DP3: now also U9.7 (DP3)
- net DPU: now also U9.16 (DPU)
- net GND: now also C20.2, C21.2, C22.2, C23.2, R14.2, U9.1 (GND), U9.12 (GND), U9.28 (GND)
- net HUB_XIN: now also U9.3 (XI)
- net HUB_XOUT: now also U9.2 (XO)
- new net: R14.1, U9.19 (PSELF)
- new net OVCUR: U9.26 (OVCUR#)
- new net PWREN: U9.25 (PWREN#)
- no-connect marks 15 -> 11
Other:
- note added: "1uF near pin 13 10uF + 0.1uF near pin 21"
- moved on the sheet: C3, C4, Y1
