File: pcb-v3/pcb-v3.kicad_pcb (KiCad board)
At the start: 2 copper layers, 312.7 x 128.6 mm, 209 parts, among them J1 Conn_01x05, J2 USB_C_Receptacle_USB2.0, SW1 SW_Push, SW2 SW_Push, U1 RP2040, U2 W25Q128JVS, U3 XC6206P332MR, X1 12MHz

Commit message: feat: attempt at routing rows
Routing:
- net ROW1: track 0.00 -> 292.6 mm
- net ROW2: track 0.00 -> 287.9 mm
- net ROW3: track 0.00 -> 284.2 mm
- net ROW0: track 0.00 -> 277.9 mm
- net ROW4: track 0.00 -> 263.1 mm
- net ROW5: track 0.00 -> 231.2 mm
